Commit message: Update to ros-gz from gazebo-ros

File: src/my_robot_description/urdf/my_robot.urdf.xacro (robot description, xacro)
@@ -217,200 +217,15 @@
     <origin xyz="0 0 ${imu_z_offset}" rpy="0 0 0"/>
   </joint>
-  <!-- Gazebo Plugins -->
-  <!-- Differential Drive -->
-  <gazebo>
-    <plugin name="differential_drive_controller" filename="libgazebo_ros_diff_drive.so">
-      <ros>
-        <namespace>/</namespace>
-        <!-- <remapping>cmd_vel:=cmd_demo</remapping> -->
-        <!-- <remapping>odom:=odom_demo</remapping> -->
-      </ros>
-      <left_joint>wheel_left_joint</left_joint>
-      <right_joint>wheel_right_joint</right_joint>
-      <wheel_separation>${wheel_separation}</wheel_separation>
-      <wheel_diameter>${wheel_diameter}</wheel_diameter>
-      <max_wheel_torque>20</max_wheel_torque>
-      <max_wheel_acceleration>1.0</max_wheel_acceleration>
-      <odometry_frame>odom</odometry_frame>
-      <robot_base_frame>base_link</robot_base_frame>
-      <publish_odom>true</publish_odom>
-      <publish_odom_tf>true</publish_odom_tf>
-      <publish_wheel_tf>false</publish_wheel_tf> <!-- Often handled by robot_state_publisher -->
-    </plugin>
-  </gazebo>
-  <!-- Front Depth Camera -->
-  <gazebo reference="camera_front_link">
-    <sensor type="depth" name="front_depth_camera_sensor">
-      <always_on>true</always_on>
-      <update_rate>15.0</update_rate>
-      <camera name="camera_front">
-        <horizontal_fov>${60.0*PI/180.0}</horizontal_fov>
-        <image>
-          <width>640</width>
-          <height>480</height>
-          <format>R8G8B8</format>
-        </image>
-        <clip>
-          <near>0.1</near>
-          <far>10.0</far>
-        </clip>
-      </camera>
-      <plugin name="front_camera_plugin" filename="libgazebo_ros_depth_camera.so">
-        <ros>
-            <namespace>/my_robot</namespace>
-            <remapping>image_raw:=camera_front/image_raw</remapping>
-            <remapping>camera_info:=camera_front/camera_info</remapping>
-            <remapping>points:=camera_front/points</remapping>
-        </ros>
-        <camera_name>camera_front</camera_name>
-        <frame_name>camera_front_link_optical</frame_name>
-        <hack_baseline>0.07</hack_baseline>
-        <min_depth>0.1</min_depth>
-        <max_depth>10.0</max_depth>
-        <point_cloud_cutoff>0.1</point_cloud_cutoff>
-        <point_cloud_cutoff_max>10.0</point_cloud_cutoff_max>
-      </plugin>
-    </sensor>
-    <!-- Add optical frame joint -->
-    <joint name="camera_front_optical_joint" type="fixed">
-      <parent link="camera_front_link" />
-      <child link="camera_front_link_optical" />
-      <origin xyz="0 0 0" rpy="${-PI/2} 0 ${-PI/2}"/>
-    </joint>
-    <link name="camera_front_link_optical"/>
-  </gazebo>
-  <!-- Rear Depth Camera -->
-  <gazebo reference="camera_rear_link">
-    <sensor type="depth" name="rear_depth_camera_sensor">
-      <always_on>true</always_on>
-      <update_rate>15.0</update_rate>
-      <camera name="camera_rear">
-        <horizontal_fov>${60.0*PI/180.0}</horizontal_fov>
-        <image>
-          <width>640</width>
-          <height>480</height>
-          <format>R8G8B8</format>
-        </image>
-        <clip>
-          <near>0.1</near>
-          <far>10.0</far>
-        </clip>
-      </camera>
-      <plugin name="rear_camera_plugin" filename="libgazebo_ros_depth_camera.so">
-        <ros>
-            <namespace>/my_robot</namespace>
-            <remapping>image_raw:=camera_rear/image_raw</remapping>
-            <remapping>camera_info:=camera_rear/camera_info</remapping>
-            <remapping>points:=camera_rear/points</remapping>
-        </ros>
-        <camera_name>camera_rear</camera_name>
-        <frame_name>camera_rear_link_optical</frame_name>
-        <hack_baseline>0.07</hack_baseline>
-        <min_depth>0.1</min_depth>
-        <max_depth>10.0</max_depth>
-        <point_cloud_cutoff>0.1</point_cloud_cutoff>
-        <point_cloud_cutoff_max>10.0</point_cloud_cutoff_max>
-      </plugin>
-    </sensor>
-    <!-- Add optical frame joint -->
-    <joint name="camera_rear_optical_joint" type="fixed">
-      <parent link="camera_rear_link" />
-      <child link="camera_rear_link_optical" />
-      <origin xyz="0 0 0" rpy="${-PI/2} 0 ${-PI/2}"/>
-    </joint>
-    <link name="camera_rear_link_optical"/>
-  </gazebo>
-  <!-- LiDAR -->
-  <gazebo reference="lidar_link">
-    <sensor type="ray" name="lidar_sensor">
-      <pose>0 0 0 0 0 0</pose>
-      <visualize>false</visualize>
-      <update_rate>10</update_rate>
-      <ray>
-        <scan>
-          <horizontal>
-            <samples>360</samples>
-            <resolution>1</resolution>
-            <min_angle>-${PI}</min_angle>
-            <max_angle>${PI}</max_angle>
-          </horizontal>
-        </scan>
-        <range>
-          <min>0.12</min>
-          <max>10.0</max>
-          <resolution>0.01</resolution>
-        </range>
-        <noise>
-          <type>gaussian</type>
-          <mean>0.0</mean>
-          <stddev>0.01</stddev>
-        </noise>
-      </ray>
-      <plugin name="lidar_plugin" filename="libgazebo_ros_ray_sensor.so">
-        <ros>
-            <namespace>/my_robot</namespace>
-            <remapping>~/out:=scan</remapping>
-        </ros>
-        <output_type>sensor_msgs/LaserScan</output_type>
-        <frame_name>lidar_link</frame_name>
-      </plugin>
-    </sensor>
-  </gazebo>
-  <!-- IMU -->
-  <gazebo reference="imu_link">
-    <sensor type="imu" name="imu_sensor">
-      <always_on>true</always_on>
-      <update_rate>100</update_rate>
-      <imu>
-        <angular_velocity>
-          <x>
-            <noise type="gaussian">
-              <mean>0.0</mean>
-              <stddev>2e-4</stddev>
-            </noise>
-          </x>
-          <y>
-            <noise type="gaussian">
-              <mean>0.0</mean>
-              <stddev>2e-4</stddev>
-            </noise>
-          </y>
-          <z>
-            <noise type="gaussian">
-              <mean>0.0</mean>
-              <stddev>2e-4</stddev>
-            </noise>
-          </z>
-        </angular_velocity>
-        <linear_acceleration>
-          <x>
-            <noise type="gaussian">
-              <mean>0.0</mean>
-              <stddev>1.7e-2</stddev>
-            </noise>
-          </x>
-          <y>
-            <noise type="gaussian">
-              <mean>0.0</mean>
-              <stddev>1.7e-2</stddev>
-            </noise>
-          </y>
-          <z>
-            <noise type="gaussian">
-              <mean>0.0</mean>
-              <stddev>1.7e-2</stddev>
-            </noise>
-          </z>
-        </linear_acceleration>
-      </imu>
-      <plugin name="imu_plugin" filename="libgazebo_ros_imu_sensor.so">
-        <ros>
-            <namespace>/my_robot</namespace>
-            <remapping>~/out:=imu/data</remapping>
-        </ros>
-        <initial_orientation_as_reference>false</initial_orientation_as_reference>
-        <frame_id>imu_link</frame_id> <!-- Gazebo Rosalind expects frame_id, not frame_name -->
-      </plugin>
-    </sensor>
-  </gazebo>
+  <!-- Example for DiffDrive plugin for Gazebo Sim: -->
+  <plugin name="diff_drive" filename="gz-sim-diff-drive-system">
+    <left_joint>wheel_left_joint</left_joint>
+    <right_joint>wheel_right_joint</right_joint>
+    <wheel_separation>${wheel_separation}</wheel_separation>
+    <wheel_radius>${wheel_radius}</wheel_radius>
+    <odom_publish>true</odom_publish>
+    <odom_frame>odom</odom_frame>
+    <robot_base_frame>base_link</robot_base_frame>
+    <topic>cmd_vel</topic>
+    <publish_tf>true</publish_tf>
+  </plugin>
 </robot>
